File: SIOSocket.sch (KiCad schematic (older format))
At the start: 2 parts, among them J1 Atari_SIO_Connector, J2 Conn_2Rows-13Pins

Commit message: Upgrade to KiCad 5.1 and changes to 3D printed SIO port for Atari800XL PCB Project
Parts:
- J1: symbol Atari:Atari_SIO_Connector -> SIOSocket-rescue:Atari_SIO_Connector-Atari
Changed lines of the file:
@@
 EESchema Schematic File Version 4
+LIBS:SIOSocket-cache
 EELAYER 30 0
 EELAYER END
@@
 $EndDescr
 $Comp
-L Atari:Atari_SIO_Connector J1
+L SIOSocket-rescue:Atari_SIO_Connector-Atari J1
 U 1 1 5DB821E3
 P 6400 3650
